File: helix.kicad_sch (KiCad schematic)
At the start: 44 parts, among them SW1 SW_Push_45deg, SW10 SW_Push_45deg, SW11 SW_Push_45deg, SW12 SW_Push_45deg, SW13 SW_Push_45deg, SW14 SW_Push_45deg, SW15 SW_Push_45deg, SW16 SW_Push_45deg, SW17 SW_Push_45deg, SW18 MLL1200S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

Commit message: updated
Parts:
- removed U1: Nice_Nano_V2, footprints:Nice_Nano_V2, symbol ScottoKeebs:MCU_Nice_Nano_V2
- added U1: Nice_Nano_V2, ScottoKeebs_MCU:Nice_Nano_V2, symbol Nice_Nano_V2:MCU_Nice_Nano_V2
Connections:
- net 1: now also U1.1
- net 2: now also U1.2 (0)
- net 20: now also U1.20 (21)
- net 21: now also U1.21 (3.3v)
- net 22: now also U1.22 (RST)
- net 23: now also U1.23 (GND)
- net 24: now also U1.24 (B+)
- net 3: now also U1.3 (GND)
- net 4: now also U1.4 (GND)
- net 5: now also U1.5 (2)
- net SW1: now also U1.17 (18)
- net SW11: now also U1.15 (14)
- net SW12: now also U1.18 (19)
- net SW13: now also U1.12 (9)
- net SW14: now also U1.11 (8)
- net SW15: now also U1.10 (7)
- net SW16: now also U1.14 (16)
- net SW17: now also U1.13 (10)
- net SW2: now also U1.9 (6)
- net SW3: now also U1.7 (4)
- net SW6: now also U1.16 (15)
- net SW7: now also U1.19 (20)
- net SW8: now also U1.8 (5)
- net SW9: now also U1.6 (3)
