File: helix.kicad_pcb (KiCad board)
At the start: 2 copper layers, 114.6 x 97.4 mm, 46 parts, among them SW1 SW_Push_45deg, SW10 SW_Push_45deg, SW11 SW_Push_45deg, SW12 SW_Push_45deg, SW13 SW_Push_45deg, SW14 SW_Push_45deg, SW15 SW_Push_45deg, SW16 SW_Push_45deg, SW17 SW_Push_45deg, SW18 MLL1200S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

Commit message: updated
Parts:
- removed the REF** at (67.3, 86.3)
- moved REF** 0.72 mm to (67.8, 86.8)
Other:
- board text removed: "LEFT"
- board text removed: "RIGHT"
